Commit message: fix: Reduce torque on the motors and the wheels.

File: project2_gochaseit/my_robot/urdf/my_robot.xacro (robot description, xacro)
@@ -57,5 +57,5 @@
     <pose>0 0 0 0 0 0</pose>
     <inertial>
-      <mass value="5"/>
+      <mass value="1"/>
       <origin rpy="1.5707 0 0" xyz="0.0 0 0"/>
       <inertia ixx="0.1" ixy="0" ixz="0" iyy="0.1" iyz="0" izz="0.1"/>
@@ -77,5 +77,5 @@
     <pose>0 0 0 0 0 0</pose>
     <inertial>
-      <mass value="5"/>
+      <mass value="1"/>
       <origin rpy="1.5707 0 0" xyz="0.0 0 0"/>
       <inertia ixx="0.1" ixy="0" ixz="0" iyy="0.1" iyz="0" izz="0.1"/>

Commit message: Change objects mass and increase support size (adapt joint pose to new size)

File: project2_gochaseit/my_robot/urdf/my_robot.xacro (robot description, xacro)
@@ -11,5 +11,5 @@
     <pose>0 0 0 0 0 0</pose>
     <inertial>
-      <mass value="2"/>
+      <mass value="3"/>
       <origin rpy="0 0 0" xyz="0.0 0 0"/>
       <inertia ixx="0.1" ixy="0" ixz="0" iyy="0.1" iyz="0" izz="0.1"/>
@@ -32,5 +32,5 @@
       <origin rpy="0 0 0" xyz="-0.035 0 -0.05"/>
       <geometry>
-        <sphere radius="0.005"/>
+        <sphere radius="0.01"/>
       </geometry>
     </collision>
@@ -38,5 +38,5 @@
       <origin rpy="0 0 0" xyz="-0.035 0 -0.05"/>
       <geometry>
-        <sphere radius="0.005"/>
+        <sphere radius="0.01"/>
       </geometry>
     </visual>
@@ -44,5 +44,5 @@
       <origin rpy="0 0 0" xyz="0.035 0 -0.05"/>
       <geometry>
-        <sphere radius="0.005"/>
+        <sphere radius="0.01"/>
       </geometry>
     </collision>
@@ -50,5 +50,5 @@
       <origin rpy="0 0 0" xyz="0.035 0 -0.05"/>
       <geometry>
-        <sphere radius="0.005"/>
+        <sphere radius="0.01"/>
       </geometry>
     </visual>
@@ -57,5 +57,5 @@
     <pose>0 0 0 0 0 0</pose>
     <inertial>
-      <mass value="1"/>
+      <mass value="5"/>
       <origin rpy="1.5707 0 0" xyz="0.0 0 0"/>
       <inertia ixx="0.1" ixy="0" ixz="0" iyy="0.1" iyz="0" izz="0.1"/>
@@ -77,5 +77,5 @@
     <pose>0 0 0 0 0 0</pose>
     <inertial>
-      <mass value="1"/>
+      <mass value="5"/>
       <origin rpy="1.5707 0 0" xyz="0.0 0 0"/>
       <inertia ixx="0.1" ixy="0" ixz="0" iyy="0.1" iyz="0" izz="0.1"/>
@@ -95,5 +95,5 @@
   </link>
   <joint name="left_wheel_hinge" type="continuous">
-    <origin rpy="0 0 0" xyz="0 0.062 -0.025"/>
+    <origin rpy="0 0 0" xyz="0 0.062 -0.03"/>
     <child link="left_wheel"/>
     <parent link="body"/>
@@ -103,5 +103,5 @@
   </joint>
   <joint name="right_wheel_hinge" type="continuous">
-    <origin rpy="0 0 0" xyz="0 -0.062 -0.025"/>
+    <origin rpy="0 0 0" xyz="0 -0.062 -0.03"/>
     <child link="right_wheel"/>
     <parent link="body"/>
@@ -115,5 +115,5 @@
     <pose>0 0 0 0 0 0</pose>
     <inertial>
-      <mass value="0"/>
+      <mass value="0.1"/>
       <origin rpy="0 0 0" xyz="0 0 0"/>
       <inertia ixx="1e-6" ixy="0" ixz="0" iyy="1e-6" iyz="0" izz="1e-6"/>
